File: ee242a-lab4-amp.sch (EAGLE design)
At the start: 0 parts

Commit message: PCBA sendout 1
Parts:
- added C1: CAP CER 10NF C0G 0402, rcl-modified-footprints:C-EUC0402
- added C10, C11, C4: CAP CER 100PF C0G 0402, rcl-modified-footprints:C-EUC0402
- added C12, C17: CAP CER 0.1UF 25V X7R 0603 10%, rcl-modified-footprints:C-EUC0603
- added C13, C16: CAP CER 10UF 16V X7R 0805 20%, rcl:C-EUC0805
- added C14: CAP CER 10000PF 25V X7R 0603 10%, rcl-modified-footprints:C-EUC0603
- added C15: CAP CER 15PF 25V X7R 0603 10%, rcl-modified-footprints:C-EUC0603
- added C2: CAP CER 2.4PF C0G 0402, rcl-modified-footprints:C-EUC0402
- added C3: CAP CER 8.2PF C0G 0402, rcl-modified-footprints:C-EUC0402
- added C5, C8, C9: CAP CER 10PF C0G 0402, rcl-modified-footprints:C-EUC0402
- added C6: CAP CER 2.7PF C0G 0402, rcl-modified-footprints:C-EUC0402
- added C7: CAP CER 1NF C0G 0402, rcl-modified-footprints:C-EUC0402
- added H1, H2, H3, H4: MOUNT-PAD-ROUND3.0, holes:MOUNT-PAD-ROUND3.0
- added IC1: TPS73001, ee242a-lab-components:TPS73001
- added L1: IND 20NF 0402, rcl-modified-footprints:L-EU0402
- added L2: IND 24NF 0402, rcl-modified-footprints:L-EU0402
- added Q1: BFG403W, ee242a-lab-components:BFG403W
- added R1, R3: RES SMD 1.6K OHM 1% 1/10W 0402, rcl-modified-footprints:R-EU_R0402
- added R2: RES SMD 1.4K OHM 1% 1/10W 0402, rcl-modified-footprints:R-EU_R0402
- added R4: RES SMD 51K OHM 1% 1/10W 0603, rcl-modified-footprints:R-EU_R0603
- added R5: RES SMD 30.1K OHM 1% 1/10W 0603, rcl-modified-footprints:R-EU_R0603
- added R6: 50R, rcl-modified-footprints:R-EU_R0805
- added TP1: VDD, ee242a-lab-components:KEYSTONE_5000
- added TP2: GND, ee242a-lab-components:KEYSTONE_5000
- added X1: IN, ee242a-lab-components:SMA-142-0701-881/886
- added X2: OUT, ee242a-lab-components:SMA-142-0701-881/886
- added X3: PWR, ee242a-lab-components:SMA-142-0701-881/886
Connections:
- new net BASE: C2.1, L1.2, Q1.B, R2.2
- new net COLLECTOR: C6.1, L2.2, Q1.C, R2.1
- new net EMITTER: C1.1, C4.1, C5.1, C7.1, Q1.E, R1.1, R3.1
- new net GND: C1.2, C10.2, C11.2, C12.2, C13.2, C14.2, C16.2, C17.2, C2.2, C4.2, C5.2, C7.2, C8.2, C9.2, H1.MOUNT, H2.MOUNT, H3.MOUNT, H4.MOUNT, IC1.GND, R1.2, R3.2, R5.2, TP2.P$1, X1G1.GND, X2G1.GND, X3G1.GND
- new net IN: C3.1, X1G1.1
- new net IN_C: C3.2, L1.1
- new net LDO_FB: C15.2, IC1.FB, R4.1, R5.1
- new net LDO_NR: C14.1, IC1.NR
- new net OUT: C6.2, X2G1.1
- new net PP_P3V3: C10.1, C11.1, C12.1, C13.1, C15.1, C8.1, C9.1, IC1.OUT, L2.1, R4.2, TP1.P$1
- new net PP_PVIN: R6.1, X3G1.1
- new net PP_PVIN_R: C16.1, C17.1, IC1.EN, IC1.IN, R6.2
