File: ee242a-lab4-amp.sch (EAGLE design)
At the start: 36 parts, among them IC1 TPS73001, Q1 BFG403W, X1 IN, X2 OUT, X3 PWR

Commit message: Created and ordered BOM
Parts:
- C1: value CAP CER 10NF C0G 0402 -> CAP CER 10000PF X7R 0402
- C13, C16: value CAP CER 10UF 16V X7R 0805 20% -> CAP CER 10UF 10V X7R 0805
- C15: value CAP CER 15PF 25V X7R 0603 10% -> CAP CER 15PF C0G 0603
- C7: value CAP CER 1NF C0G 0402 -> CAP CER 1000PF C0G 0402
- L1: value IND 20NF 0402 -> IND 20NH 0402
- L2: value IND 24NF 0402 -> IND 24NH 0402
Other:
- moved on the sheet: C1
