File: ee242a-lab4-amp -values2.sch (EAGLE design)
At the start: 36 parts, among them IC1 TPS73001, Q1 BFG403W, X1 IN, X2 OUT, X3 PWR

Commit message: Updated component values
Parts:
- C2: value CAP CER 2.4PF C0G 0402 -> CAP CER 2.2PF C0G 0402
- L1: value IND 20NH 0402 -> IND 26NH 0402
- L2: value IND 24NH 0402 -> IND 30NH 0402
- R2: value RES SMD 1.4K OHM 1% 1/10W 0402 -> RES SMD 1.74K OHM 1% 1/10W 0402
Other:
- note added: "Add 51R1 base res"
- note added: "Previously 1.40k"
- note added: "Previously 2.4pF"
- note added: "Previously 20nH"
- note removed: "USE 30nH, 0402 has higher SRF"
Changed lines of the file:
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@@
 <part name="C4" library="rcl-modified-footprints" deviceset="C-EU" device="C0402" package3d_urn="urn:adsk.eagle:package:23626/1" value="CAP CER 100PF C0G 0402"/>
 <part name="R3" library="rcl-modified-footprints" deviceset="R-EU_" device="R0402" package3d_urn="urn:adsk.eagle:package:23547/1" value="RES SMD 1.6K OHM 1% 1/10W 0402"/>
-<part name="R2" library="rcl-modified-footprints" deviceset="R-EU_" device="R0402" package3d_urn="urn:adsk.eagle:package:23547/1" value="RES SMD 1.4K OHM 1% 1/10W 0402"/>
-<part name="L2" library="rcl-modified-footprints" deviceset="L-EU" device="0402" package3d_urn="urn:adsk.eagle:package:23547/1" value="IND 24NH 0402"/>
-<part name="L1" library="rcl-modified-footprints" deviceset="L-EU" device="0402" package3d_urn="urn:adsk.eagle:package:23547/1" value="IND 20NH 0402"/>
-<part name="C2" library="rcl-modified-footprints" deviceset="C-EU" device="C0402" package3d_urn="urn:adsk.eagle:package:23626/1" value="CAP CER 2.4PF C0G 0402"/>
+<part name="R2" library="rcl-modified-footprints" deviceset="R-EU_" device="R0402" package3d_urn="urn:adsk.eagle:package:23547/1" value="RES SMD 1.74K OHM 1% 1/10W 0402"/>
+<part name="L2" library="rcl-modified-footprints" deviceset="L-EU" device="0402" package3d_urn="urn:adsk.eagle:package:23547/1" value="IND 30NH 0402"/>
+<part name="L1" library="rcl-modified-footprints" deviceset="L-EU" device="0402" package3d_urn="urn:adsk.eagle:package:23547/1" value="IND 26NH 0402"/>
+<part name="C2" library="rcl-modified-footprints" deviceset="C-EU" device="C0402" package3d_urn="urn:adsk.eagle:package:23626/1" value="CAP CER 2.2PF C0G 0402"/>
 <part name="C6" library="rcl-modified-footprints" deviceset="C-EU" device="C0402" package3d_urn="urn:adsk.eagle:package:23626/1" value="CAP CER 2.7PF C0G 0402"/>
 <part name="C3" library="rcl-modified-footprints" deviceset="C-EU" device="C0402" package3d_urn="urn:adsk.eagle:package:23626/1" value="CAP CER 8.2PF C0G 0402"/>
@@
 <sheet>
 <plain>
-<text x="129.54" y="121.92" size="1.778" layer="98">USE 30nH, 0402 has higher SRF</text>
+<text x="116.84" y="58.42" size="0.8128" layer="98">Previously 2.4pF</text>
+<text x="104.14" y="88.9" size="0.8128" layer="98">Previously 1.40k</text>
+<text x="116.84" y="76.2" size="0.8128" layer="98">Add 51R1 base res</text>
+<text x="91.44" y="73.66" size="0.8128" layer="98">Previously 20nH</text>
 </plain>
 <instances>
