File: ee242a-lab4-amp.brd (EAGLE design)
At the start: 38.1 x 38.1 mm, 36 parts, among them IC1 TPS73001, Q1 BFG403W, X1 IN, X2 OUT, X3 PWR

Commit message: Created and ordered BOM
Parts:
- C1: value CAP CER 10NF C0G 0402 -> CAP CER 10000PF X7R 0402
- C13, C16: value CAP CER 10UF 16V X7R 0805 20% -> CAP CER 10UF 10V X7R 0805
- C15: value CAP CER 15PF 25V X7R 0603 10% -> CAP CER 15PF C0G 0603
- C7: value CAP CER 1NF C0G 0402 -> CAP CER 1000PF C0G 0402
- L1: value IND 20NF 0402 -> IND 20NH 0402
- L2: value IND 24NF 0402 -> IND 24NH 0402
Changed lines of the file:
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@@
 <?xml version="1.0" encoding="utf-8"?>
 <!DOCTYPE eagle SYSTEM "eagle.dtd">
-<eagle version="9.2.2">
+<eagle version="9.0.1">
 <drawing>
 <settings>
@@
 <param name="checkStop" value="0"/>
 <param name="checkValues" value="0"/>
-<param name="checkNames" value="1"/>
-<param name="checkWireStubs" value="1"/>
-<param name="checkPolygonWidth" value="0"/>
 <param name="useDiameter" value="13"/>
 <param name="maxErrors" value="50"/>
@@
 <attribute name="NAME" x="14.12875" y="23.33625" size="0.8128" layer="25" font="vector" ratio="16" rot="R180"/>
 </element>
-<element name="C7" library="rcl-modified-footprints" package="C0402" package3d_urn="urn:adsk.eagle:package:23626/1" value="CAP CER 1NF C0G 0402" x="17.145" y="21.74875" smashed="yes">
+<element name="C7" library="rcl-modified-footprints" package="C0402" package3d_urn="urn:adsk.eagle:package:23626/1" value="CAP CER 1000PF C0G 0402" x="17.145" y="21.74875" smashed="yes">
 <attribute name="NAME" x="14.12875" y="21.11375" size="0.8128" layer="25" font="vector" ratio="16" rot="R180"/>
 </element>
-<element name="C1" library="rcl-modified-footprints" package="C0402" package3d_urn="urn:adsk.eagle:package:23626/1" value="CAP CER 10NF C0G 0402" x="19.05" y="25.7175" smashed="yes" rot="R90">
+<element name="C1" library="rcl-modified-footprints" package="C0402" package3d_urn="urn:adsk.eagle:package:23626/1" value="CAP CER 10000PF X7R 0402" x="19.05" y="25.7175" smashed="yes" rot="R90">
 <attribute name="NAME" x="20.79625" y="25.7175" size="0.8128" layer="25" font="vector" ratio="16"/>
 </element>
@@
 <attribute name="NAME" x="11.27125" y="24.765" size="0.8128" layer="25" font="vector" ratio="16"/>
 </element>
-<element name="L2" library="rcl-modified-footprints" package="R0402" package3d_urn="urn:adsk.eagle:package:23547/1" value="IND 24NF 0402" x="19.685" y="22.225" smashed="yes" rot="R90">
+<element name="L2" library="rcl-modified-footprints" package="R0402" package3d_urn="urn:adsk.eagle:package:23547/1" value="IND 24NH 0402" x="19.685" y="22.225" smashed="yes" rot="R90">
 <attribute name="NAME" x="20.32" y="21.2725" size="0.8128" layer="25" font="vector" ratio="16"/>
 </element>
-<element name="L1" library="rcl-modified-footprints" package="R0402" package3d_urn="urn:adsk.eagle:package:23547/1" value="IND 20NF 0402" x="14.12875" y="24.13" smashed="yes">
+<element name="L1" library="rcl-modified-footprints" package="R0402" package3d_urn="urn:adsk.eagle:package:23547/1" value="IND 20NH 0402" x="14.12875" y="24.13" smashed="yes">
 <attribute name="NAME" x="13.17625" y="24.765" size="0.8128" layer="25" font="vector" ratio="16"/>
 </element>
@@
 <attribute name="NAME" x="20.6375" y="10.00125" size="0.8128" layer="25" font="vector" ratio="16"/>
 </element>
-<element name="C15" library="rcl-modified-footprints" package="C0603" package3d_urn="urn:adsk.eagle:package:23616/2" value="CAP CER 15PF 25V X7R 0603 10%" x="16.8275" y="13.81125" smashed="yes" rot="R270">
+<element name="C15" library="rcl-modified-footprints" package="C0603" package3d_urn="urn:adsk.eagle:package:23616/2" value="CAP CER 15PF C0G 0603" x="16.8275" y="13.81125" smashed="yes" rot="R270">
 <attribute name="NAME" x="14.44625" y="14.76375" size="0.8128" layer="25" font="vector" ratio="16" rot="R180"/>
 </element>
@@
 <attribute name="NAME" x="21.59" y="16.8275" size="0.8128" layer="25" font="vector" ratio="16"/>
 </element>
-<element name="C13" library="rcl" package="C0805" value="CAP CER 10UF 16V X7R 0805 20%" x="16.1925" y="16.98625" smashed="yes" rot="R180">
+<element name="C13" library="rcl" package="C0805" value="CAP CER 10UF 10V X7R 0805" x="16.1925" y="16.98625" smashed="yes" rot="R180">
 <attribute name="NAME" x="14.2875" y="17.78" size="0.8128" layer="25" font="vector" ratio="16" rot="R180"/>
 </element>
@@
 <attribute name="VALUE" x="12.7" y="1.27" size="1.27" layer="27" font="vector" ratio="16" rot="R90"/>
 </element>
-<element name="C16" library="rcl" package="C0805" value="CAP CER 10UF 16V X7R 0805 20%" x="15.71625" y="10.4775" smashed="yes" rot="R180">
+<element name="C16" library="rcl" package="C0805" value="CAP CER 10UF 10V X7R 0805" x="15.71625" y="10.4775" smashed="yes" rot="R180">
 <attribute name="NAME" x="13.81125" y="11.27125" size="0.8128" layer="25" font="vector" ratio="16" rot="R180"/>
 </element>
@@
 </signal>
 </signals>
-<mfgpreviewcolors>
-<mfgpreviewcolor name="soldermaskcolor" color="0xC8008000"/>
-<mfgpreviewcolor name="silkscreencolor" color="0xFFFEFEFE"/>
-<mfgpreviewcolor name="backgroundcolor" color="0xFF282828"/>
-<mfgpreviewcolor name="coppercolor" color="0xFFFFBF00"/>
-<mfgpreviewcolor name="substratecolor" color="0xFF786E46"/>
-</mfgpreviewcolors>
 </board>
 </drawing>
