File: ee242a-lab4-amp2.brd (EAGLE design)
At the start: 38.1 x 38.1 mm, 36 parts, among them IC1 TPS73001, Q1 BFG403W, X1 IN, X2 OUT, X3 PWR

Commit message: Cleanup
Parts:
- C2: value CAP CER 2.4PF C0G 0402 -> CAP CER 2.2PF C0G 0402
- L1: value IND 20NH 0402 -> IND 26NH 0402
- L2: value IND 24NH 0402 -> IND 30NH 0402
- R2: value RES SMD 1.4K OHM 1% 1/10W 0402 -> RES SMD 2.2K OHM 1% 1/10W 0402
Changed lines of the file:
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@@
 <attribute name="NAME" x="21.2725" y="23.8125" size="0.8128" layer="25" font="vector" ratio="16"/>
 </element>
-<element name="C2" library="rcl-modified-footprints" package="C0402" package3d_urn="urn:adsk.eagle:package:23626/1" value="CAP CER 2.4PF C0G 0402" x="15.71625" y="24.60625" smashed="yes" rot="R90">
+<element name="C2" library="rcl-modified-footprints" package="C0402" package3d_urn="urn:adsk.eagle:package:23626/1" value="CAP CER 2.2PF C0G 0402" x="15.71625" y="24.60625" smashed="yes" rot="R90">
 <attribute name="NAME" x="16.1925" y="26.51125" size="0.8128" layer="25" font="vector" ratio="16" rot="R180"/>
 </element>
@@
 <attribute name="NAME" x="11.27125" y="24.765" size="0.8128" layer="25" font="vector" ratio="16"/>
 </element>
-<element name="L2" library="rcl-modified-footprints" package="R0402" package3d_urn="urn:adsk.eagle:package:23547/1" value="IND 24NH 0402" x="19.685" y="22.225" smashed="yes" rot="R90">
+<element name="L2" library="rcl-modified-footprints" package="R0402" package3d_urn="urn:adsk.eagle:package:23547/1" value="IND 30NH 0402" x="19.685" y="22.225" smashed="yes" rot="R90">
 <attribute name="NAME" x="20.32" y="21.2725" size="0.8128" layer="25" font="vector" ratio="16"/>
 </element>
-<element name="L1" library="rcl-modified-footprints" package="R0402" package3d_urn="urn:adsk.eagle:package:23547/1" value="IND 20NH 0402" x="14.12875" y="24.13" smashed="yes">
+<element name="L1" library="rcl-modified-footprints" package="R0402" package3d_urn="urn:adsk.eagle:package:23547/1" value="IND 26NH 0402" x="14.12875" y="24.13" smashed="yes">
 <attribute name="NAME" x="13.17625" y="24.765" size="0.8128" layer="25" font="vector" ratio="16"/>
 </element>
@@
 <attribute name="NAME" x="14.12875" y="22.225" size="0.8128" layer="25" font="vector" ratio="16" rot="R180"/>
 </element>
-<element name="R2" library="rcl-modified-footprints" package="R0402" package3d_urn="urn:adsk.eagle:package:23547/1" value="RES SMD 1.4K OHM 1% 1/10W 0402" x="17.30375" y="25.24125" smashed="yes" rot="R180">
+<element name="R2" library="rcl-modified-footprints" package="R0402" package3d_urn="urn:adsk.eagle:package:23547/1" value="RES SMD 2.2K OHM 1% 1/10W 0402" x="17.30375" y="25.24125" smashed="yes" rot="R180">
 <attribute name="NAME" x="16.66875" y="25.87625" size="0.8128" layer="25" font="vector" ratio="16"/>
 </element>
